File: Hardware Design and System Updates/Main-Unit-and-PSU/main-unit-psu.sch (EAGLE design)
At the start: 5 parts, among them U1 BA033CC0FP-E2TO252-3_ROM

Commit message: Integraded members parts
Parts:
- added B1: KMB23S, rectifier:B-DIL
- added C1: 470 uF, rcl:C-US050-024X044
- added C2: 0.1 uF, rcl:C-US050-024X044
- added D1, D3: 1N4004, diode:1N4004
- added D2: NZX22C,133, diode:ZENER-DIODEDO41Z10
- added DC2: K7803-500R3, dc-dc-converter:NME
- added DC3: R-78W9.0-0.5, dc-dc-converter:NME
- added E1: HM-10-BOARD, HM-10:HM-10-BOARD
- added TR1: TCT50-01E07AB, trafo:EE20-1
- added U2: BA033CC0FP-E2TO252-3_ROM, 2023-03-08_12-17-23_Library:BA033CC0FP-E2TO252-3_ROM
- added U3: MSP430FR2110IPW16, MSP430FR2110:MSP430FR2110IPW16
Connections:
- removed net N$6 (its old number): BT2.-, DC1.+VIN
- new net N$10: E1.UART_TX, U3.P1.6/UCA0RXD/UCA0SOMI/TB0.1/TDI/TCLK/A6
- new net N$11: D1.A, DC2.+VIN, DC3.+VOUT
- new net N$12: C3.1, E1.+3.3V, U1.OUT, U3.DVCC
- new net N$13: E1.UART_RX, U3.P1.7/UCA0TXD/UCA0SIMO/TB0.2/TDO/A7/VREF+
- new net N$2: B1.AC2, TR1.S3
- new net N$3: C2.1, U2.OUT, U3.P1.1/UCA0CLK/ACLK/C1/A1
- new net N$5: D1.C, D3.C, DC1.+VIN
- new net N$7: BT2.-, D3.A
- new net N$8: B1.+, C1.1, D2.C, DC3.+VIN
- new net N$9: DC2.+VOUT, U2.VCC
- net 0: now also B1.-, C1.2, C2.2, D2.A, DC2.-VIN, DC2.-VOUT, DC3.-VIN, DC3.-VOUT, E1.GND, U3.DVSS
- net N$1: now also B1.AC1, TR1.S4; no longer C3.1, U1.OUT
Other:
- moved on the sheet: BT1, BT2, C3, DC1, U1
