File: PROTOTYPE INTEGRATION and System Updates/System-Schematic-Diagrams/Main-Unit-and-PSU/main-unit-psu.sch (EAGLE design)
At the start: 26 parts, among them U1 BA033CC0FP-E2TO252-3_ROM, U2 BA033CC0FP-E2TO252-3_ROM, U3 MSP430FR2110IPW16, U4 MCP6022-I/P, U5 TMP36GT9ZT_3_ADI, U6 L7805CV, U7 RAC03-12SKRAC03-K_RCP

Commit message: Updated Schematics and BOM
Parts:
- removed C4: 0.1 uF, rcl:C-US050-024X044
- removed DC4: TSR 1-2450, dc-dc-converter:NME
- removed E1: HM-10-BOARD, HM-10:HM-10-BOARD
- removed R4: 620 Ohm, rcl:R-US_0204/7
- removed R5: 39 Ohm, rcl:R-US_0204/7
- removed R6: 5.1 Ohm, rcl:R-US_0204/7
- removed R7: 1 kOhm, rcl:R-US_0204/7
- removed U4: MCP6022-I/P, MCP6022-I_P:MCP6022-I/P
- removed U5: TMP36GT9ZT_3_ADI, 2023-03-28_14-12-25_Library:TMP36GT9ZT_3_ADI
- removed U6: L7805CV, 2023-03-08_12-17-23_Library:BA033CC0FP-E2TO252-3_ROM
- added R2: 1 KOhm, rcl:R-US_0207/2V
- R1: value 65 Ohm -> 1 KOhm
- R3: value 100 Ohm -> 1 KOhm
Connections:
- removed net +5V: DC4.+VIN
- removed net N$14: R7.1, U5.VOUT
- removed net N$18: R5.1, R6.2
- removed net N$19: R4.1, R5.2
- removed net N$20: R6.1, U3.P1.2/UCA0RXD/UCA0SOMI/TB0TRG/C2/A2/VEREF-, U4.VOUTA
- removed net N$21: R4.2, R7.2, U4.VINA+
- removed net VCC: U4.VDD
- net 0: now also R2.1; no longer C4.2, DC4.-VIN, DC4.-VOUT, E1.GND, U4.VSS, U5.GND
- net N$10: no longer E1.UART_TX
- net N$13: no longer E1.UART_RX
- net N$3: now also R2.2
- net N$4: no longer DC4.+VOUT, U6.VCC
- net VCC1: no longer C4.1, E1.+3.3V, U5.+VS, U6.OUT
