File: PROTOTYPE INTEGRATION and System Updates/System-Schematic-Diagrams/Sub-Unit/SUB-UNIT.sch (EAGLE design)
At the start: 13 parts, among them U1 MSP430FR2000IPW16PW16_TEX, U3 L7805CV, U4 TMP36GT9ZT_3_ADI, U5 MCP6022-I/P

Commit message: Updated Schematics and BOM
Parts:
- removed C3: 0.1 uF, rcl:C-US050-024X044
- removed DC1: TSR 1-2450, dc-dc-converter:NME
- removed E1: HM-10-BOARD, HM-10 Bluetooth Module:HM-10-BOARD
- removed U3: L7805CV, 2023-03-08_12-17-23_Library:BA033CC0FP-E2TO252-3_ROM
- R1: value 68 Ohms -> 1 KOhms
Connections:
- removed net +5V: DC1.+VIN
- net 0: no longer C3.2, DC1.-VIN, DC1.-VOUT
- net GND: no longer E1.GND
- net N$12: no longer C3.1, E1.+3.3V, U3.OUT
- net N$2: no longer E1.UART_TX
- net N$3: now also U1.P1.3/UCA0TXD/UCA0SIMO/C3/A3; no longer E1.UART_RX, U1.P1.7/_/TB0.2/TDO/A7_UCA0TXD/UCA0SIMO_/VREF+
- net N$4: no longer DC1.+VOUT, U3.VCC
Changed lines of the file:
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@@
 </classes>
 <parts>
-<part name="E1" library="HM-10 Bluetooth Module" deviceset="HM-10" device="-BOARD"/>
 <part name="LED1" library="Lumex SSL-LX3052ID RED LED" deviceset="SSL-LX3052ID" device=""/>
-<part name="R1" library="adafruit" deviceset="R-US_" device="0204/5" value="68 Ohms"/>
+<part name="R1" library="adafruit" deviceset="R-US_" device="0204/5" value="1 KOhms"/>
 <part name="U1" library="MSP430FR2000 Sub-Unit" deviceset="MSP430FR2000IPW16" device="PW16_TEX"/>
 <part name="SUPPLY2" library="supply2" library_urn="urn:adsk.eagle:library:372" deviceset="GND" device=""/>
-<part name="SUPPLY1" library="supply2" library_urn="urn:adsk.eagle:library:372" deviceset="GND" device=""/>
 <part name="SUPPLY3" library="supply2" library_urn="urn:adsk.eagle:library:372" deviceset="GND" device=""/>
 <part name="P+1" library="supply1" library_urn="urn:adsk.eagle:library:371" deviceset="VCC" device=""/>
@@
 <part name="U4" library="2023-03-28_14-12-25_Library" deviceset="TMP36GT9Z" device="T_3_ADI"/>
 <part name="X_3" library="ngspice-simulation" library_urn="urn:adsk.eagle:library:527439" deviceset="GND" device=""/>
-<part name="DC1" library="dc-dc-converter" library_urn="urn:adsk.eagle:library:208" deviceset="NME" device="" package3d_urn="urn:adsk.eagle:package:12313/1" value="TSR 1-2450"/>
-<part name="X_6" library="ngspice-simulation" library_urn="urn:adsk.eagle:library:527439" deviceset="GND" device=""/>
-<part name="U3" library="2023-03-08_12-17-23_Library" deviceset="BA033CC0FP-E2" device="TO252-3_ROM" value="L7805CV"/>
-<part name="X_8" library="ngspice-simulation" library_urn="urn:adsk.eagle:library:527439" deviceset="GND" device=""/>
-<part name="C3" library="rcl" library_urn="urn:adsk.eagle:library:334" deviceset="C-US" device="050-024X044" package3d_urn="urn:adsk.eagle:package:23643/1" value="0.1 uF"/>
-<part name="X_10" library="ngspice-simulation" library_urn="urn:adsk.eagle:library:527439" deviceset="GND" device=""/>
-<part name="P+3" library="supply1" library_urn="urn:adsk.eagle:library:371" deviceset="+5V" device="" value="+9V"/>
 <part name="U5" library="MCP6022-I_P" deviceset="MCP6022-I/P" device=""/>
 </parts>
@@
 </plain>
 <instances>
-<instance part="E1" gate="G$1" x="-109.22" y="132.08" smashed="yes">
-<attribute name="NAME" x="-93.98" y="86.36" size="1.6764" layer="94" rot="R90"/>
-</instance>
 <instance part="LED1" gate="A" x="-279.4" y="142.24" smashed="yes">
 <attribute name="VALUE" x="-283.2862" y="132.8928" size="3.4798" layer="96" ratio="10" rot="SR0"/>
@@
 <instance part="SUPPLY2" gate="GND" x="-259.08" y="139.7" smashed="yes">
 <attribute name="VALUE" x="-260.985" y="136.525" size="1.778" layer="96"/>
-</instance>
-<instance part="SUPPLY1" gate="GND" x="-119.38" y="83.82" smashed="yes">
-<attribute name="VALUE" x="-121.285" y="80.645" size="1.778" layer="96"/>
 </instance>
 <instance part="SUPPLY3" gate="GND" x="-302.26" y="99.06" smashed="yes">
@@
 </instance>
 <instance part="X_3" gate="G$1" x="-264.16" y="38.1" smashed="yes"/>
-<instance part="DC1" gate="G$1" x="-226.06" y="22.86" smashed="yes">
-<attribute name="NAME" x="-236.22" y="28.575" size="1.778" layer="95"/>
-<attribute name="VALUE" x="-236.22" y="12.7" size="1.778" layer="96"/>
-</instance>
-<instance part="X_6" gate="G$1" x="-241.3" y="15.24" smashed="yes"/>
-<instance part="U3" gate="A" x="-203.2" y="25.4" smashed="yes">
-<attribute name="NAME" x="-185.0654" y="34.5186" size="2.083" layer="95" ratio="6"/>
-<attribute name="VALUE" x="-185.7048" y="31.9786" size="2.083" layer="96" ratio="6"/>
-</instance>
-<instance part="X_8" gate="G$1" x="-198.12" y="10.16" smashed="yes"/>
-<instance part="C3" gate="G$1" x="-154.94" y="20.32" smashed="yes">
-<attribute name="NAME" x="-153.924" y="20.955" size="1.778" layer="95"/>
-<attribute name="VALUE" x="-153.924" y="16.129" size="1.778" layer="96"/>
-</instance>
-<instance part="X_10" gate="G$1" x="-154.94" y="12.7" smashed="yes"/>
-<instance part="P+3" gate="1" x="-256.54" y="35.56" smashed="yes">
-<attribute name="VALUE" x="-259.08" y="30.48" size="1.778" layer="96" rot="R90"/>
-</instance>
 <instance part="U5" gate="A" x="-193.04" y="60.96" smashed="yes">
 <attribute name="NAME" x="-205.74" y="74.66" size="2.0828" layer="95" ratio="10" rot="SR0"/>
@@
 </segment>
 <segment>
-<pinref part="E1" gate="G$1" pin="GND"/>
-<wire x1="-114.3" y1="91.44" x2="-119.38" y2="91.44" width="0.1524" layer="91"/>
-<pinref part="SUPPLY1" gate="GND" pin="GND"/>
-<wire x1="-119.38" y1="91.44" x2="-119.38" y2="86.36" width="0.1524" layer="91"/>
-</segment>
-<segment>
 <pinref part="U1" gate="A" pin="DVSS"/>
 <wire x1="-299.72" y1="109.22" x2="-302.26" y2="109.22" width="0.1524" layer="91"/>
@@
 </segment>
 </net>
-<net name="N$2" class="0">
-<segment>
-<pinref part="E1" gate="G$1" pin="UART_TX"/>
-<wire x1="-114.3" y1="121.92" x2="-119.38" y2="121.92" width="0.1524" layer="91"/>
-<wire x1="-119.38" y1="121.92" x2="-119.38" y2="111.76" width="0.1524" layer="91"/>
-<pinref part="U1" gate="A" pin="P1.6/UCA0RXD/UCA0SOMI/TB0.1/TDI/TCLK/A6"/>
-<wire x1="-119.38" y1="111.76" x2="-121.92" y2="111.76" width="0.1524" layer="91"/>
-</segment>
-</net>
-<net name="N$3" class="0">
-<segment>
-<pinref part="E1" gate="G$1" pin="UART_RX"/>
-<wire x1="-114.3" y1="119.38" x2="-116.84" y2="119.38" width="0.1524" layer="91"/>
-<wire x1="-116.84" y1="119.38" x2="-116.84" y2="109.22" width="0.1524" layer="91"/>
-<pinref part="U1" gate="A" pin="P1.7/_/TB0.2/TDO/A7_UCA0TXD/UCA0SIMO_/VREF+"/>
-<wire x1="-116.84" y1="109.22" x2="-121.92" y2="109.22" width="0.1524" layer="91"/>
-</segment>
-</net>
 <net name="N$4" class="0">
 <segment>
@@
 <pinref part="R1" gate="G$1" pin="2"/>
 <wire x1="-299.72" y1="121.92" x2="-299.72" y2="142.24" width="0.1524" layer="91"/>
-</segment>
-<segment>
-<pinref part="DC1" gate="G$1" pin="+VOUT"/>
-<wire x1="-213.36" y1="25.4" x2="-200.66" y2="25.4" width="0.1524" layer="91"/>
-<label x="-213.36" y="25.4" size="1.778" layer="95"/>
-<pinref part="U3" gate="A" pin="VCC"/>
 </segment>
 </net>
@@
 </segment>
 <segment>
-<pinref part="X_6" gate="G$1" pin="0"/>
-<pinref part="DC1" gate="G$1" pin="-VIN"/>
-<wire x1="-241.3" y1="15.24" x2="-241.3" y2="20.32" width="0.1524" layer="91"/>
-<wire x1="-241.3" y1="20.32" x2="-238.76" y2="20.32" width="0.1524" layer="91"/>
-</segment>
-<segment>
-<pinref part="DC1" gate="G$1" pin="-VOUT"/>
-<wire x1="-213.36" y1="20.32" x2="-213.36" y2="15.24" width="0.1524" layer="91"/>
-<wire x1="-213.36" y1="15.24" x2="-198.12" y2="15.24" width="0.1524" layer="91"/>
-<pinref part="X_8" gate="G$1" pin="0"/>
-<wire x1="-198.12" y1="10.16" x2="-198.12" y2="15.24" width="0.1524" layer="91"/>
-</segment>
-<segment>
-<pinref part="X_10" gate="G$1" pin="0"/>
-<pinref part="C3" gate="G$1" pin="2"/>
-<wire x1="-154.94" y1="12.7" x2="-154.94" y2="15.24" width="0.1524" layer="91"/>
-</segment>
-<segment>
 <pinref part="U5" gate="A" pin="VSS"/>
 <wire x1="-175.26" y1="50.8" x2="-172.72" y2="50.8" width="0.1524" layer="91"/>
@@
 <wire x1="-215.9" y1="45.72" x2="-215.9" y2="66.04" width="0.1524" layer="91"/>
 <wire x1="-215.9" y1="66.04" x2="-210.82" y2="66.04" width="0.1524" layer="91"/>
-</segment>
-<segment>
-<wire x1="-160.02" y1="25.4" x2="-154.94" y2="25.4" width="0.1524" layer="91"/>
-<label x="-157.48" y="27.94" size="1.778" layer="95"/>
-<pinref part="U3" gate="A" pin="OUT"/>
-<pinref part="C3" gate="G$1" pin="1"/>
-<wire x1="-154.94" y1="22.86" x2="-154.94" y2="25.4" width="0.1524" layer="91"/>
-<pinref part="E1" gate="G$1" pin="+3.3V"/>
-<wire x1="-114.3" y1="93.98" x2="-114.3" y2="25.4" width="0.1524" layer="91"/>
-<wire x1="-114.3" y1="25.4" x2="-154.94" y2="25.4" width="0.1524" layer="91"/>
-<junction x="-154.94" y="25.4"/>
 </segment>
 </net>
@@
 </segment>
 </net>
-<net name="+5V" class="0">
-<segment>
-<pinref part="DC1" gate="G$1" pin="+VIN"/>
-<wire x1="-256.54" y1="25.4" x2="-238.76" y2="25.4" width="0.1524" layer="91"/>
-<pinref part="P+3" gate="1" pin="+5V"/>
-<wire x1="-256.54" y1="25.4" x2="-256.54" y2="33.02" width="0.1524" layer="91"/>
-</segment>
-</net>
+<net name="N$2" class="0">
+<segment>
+<pinref part="U1" gate="A" pin="P1.6/UCA0RXD/UCA0SOMI/TB0.1/TDI/TCLK/A6"/>
+<wire x1="-121.92" y1="111.76" x2="-111.76" y2="111.76" width="0.1524" layer="91"/>
+</segment>
+</net>
+<net name="N$3" class="0">
+<segment>
+<pinref part="U1" gate="A" pin="P1.3/UCA0TXD/UCA0SIMO/C3/A3"/>
+<wire x1="-121.92" y1="119.38" x2="-111.76" y2="119.38" width="0.1524" layer="91"/>
+</segment>
+</net>
