File: PROTOTYPE INTEGRATION and System Updates/System-Schematic-Diagrams/Sub-Unit-and-PSU/sub-unit-and-psu.sch (EAGLE design)
At the start: 18 parts, among them U1 BA033CC0FP-E2TO252-3_ROM, U2 MSP430FR2000IPW16PW16_TEX, U3 MCP6022-I/P, U4 TMP36GT9ZT_3_ADI, U5 L7805CV

Commit message: Updated Schematics and BOM
Parts:
- removed C1: 0.1 uF, rcl:C-US050-024X044
- removed DC2: TSR 1-2450, dc-dc-converter:NME
- removed E1: HM-10-BOARD, HM-10 Bluetooth Module:HM-10-BOARD
- removed U5: L7805CV, 2023-03-08_12-17-23_Library:BA033CC0FP-E2TO252-3_ROM
- R1: value 68 Ohms -> 1 KOhm
Connections:
- removed net N$12: C1.1, E1.+3.3V, U5.OUT
- new net N$10: U2.P2.1/TB0.2
- net 0: no longer C1.2, DC2.-VIN, DC2.-VOUT
- net GND: no longer E1.GND
- net N$15: now also U2.P1.2/UCA0RXD/UCA0SOMI/TB0TRG/C2/A2/VEREF-; no longer U2.P2.1/TB0.2
- net N$4: no longer DC2.+VOUT, U5.VCC
- net N$5: no longer E1.UART_TX
- net N$6: no longer DC2.+VIN
- net N$7: no longer E1.UART_RX
Changed lines of the file:
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@@
 <part name="C3" library="rcl" library_urn="urn:adsk.eagle:library:334" deviceset="C-US" device="050-024X044" package3d_urn="urn:adsk.eagle:package:23643/1" value="0.1 uF"/>
 <part name="X_10" library="ngspice-simulation" library_urn="urn:adsk.eagle:library:527439" deviceset="GND" device=""/>
-<part name="E1" library="HM-10 Bluetooth Module" deviceset="HM-10" device="-BOARD"/>
 <part name="LED1" library="Lumex SSL-LX3052ID RED LED" deviceset="SSL-LX3052ID" device=""/>
-<part name="R1" library="adafruit" deviceset="R-US_" device="0204/5" value="68 Ohms"/>
+<part name="R1" library="adafruit" deviceset="R-US_" device="0204/5" value="1 KOhm"/>
 <part name="U2" library="MSP430FR2000 Sub-Unit" deviceset="MSP430FR2000IPW16" device="PW16_TEX"/>
 <part name="SUPPLY2" library="supply2" library_urn="urn:adsk.eagle:library:372" deviceset="GND" device=""/>
-<part name="SUPPLY1" library="supply2" library_urn="urn:adsk.eagle:library:372" deviceset="GND" device=""/>
 <part name="SUPPLY3" library="supply2" library_urn="urn:adsk.eagle:library:372" deviceset="GND" device=""/>
 <part name="P+2" library="supply1" library_urn="urn:adsk.eagle:library:371" deviceset="VCC" device="" value="3.3V"/>
@@
 <part name="U4" library="2023-03-28_14-12-25_Library" deviceset="TMP36GT9Z" device="T_3_ADI"/>
 <part name="X_3" library="ngspice-simulation" library_urn="urn:adsk.eagle:library:527439" deviceset="GND" device=""/>
-<part name="DC2" library="dc-dc-converter" library_urn="urn:adsk.eagle:library:208" deviceset="NME" device="" package3d_urn="urn:adsk.eagle:package:12313/1" value="TSR 1-2450"/>
-<part name="X_5" library="ngspice-simulation" library_urn="urn:adsk.eagle:library:527439" deviceset="GND" device=""/>
-<part name="U5" library="2023-03-08_12-17-23_Library" deviceset="BA033CC0FP-E2" device="TO252-3_ROM" value="L7805CV"/>
-<part name="X_8" library="ngspice-simulation" library_urn="urn:adsk.eagle:library:527439" deviceset="GND" device=""/>
-<part name="C1" library="rcl" library_urn="urn:adsk.eagle:library:334" deviceset="C-US" device="050-024X044" package3d_urn="urn:adsk.eagle:package:23643/1" value="0.1 uF"/>
-<part name="X_7" library="ngspice-simulation" library_urn="urn:adsk.eagle:library:527439" deviceset="GND" device=""/>
 <part name="U3" library="MCP6022-I_P" deviceset="MCP6022-I/P" device=""/>
 </parts>
@@
 </instance>
 <instance part="X_10" gate="G$1" x="233.68" y="134.62" smashed="yes"/>
-<instance part="E1" gate="G$1" x="449.58" y="142.24" smashed="yes">
-<attribute name="NAME" x="464.82" y="96.52" size="1.6764" layer="94" rot="R90"/>
-</instance>
 <instance part="LED1" gate="A" x="279.4" y="152.4" smashed="yes">
 <attribute name="VALUE" x="275.5138" y="143.0528" size="3.4798" layer="96" ratio="10" rot="SR0"/>
@@
 <instance part="SUPPLY2" gate="GND" x="299.72" y="149.86" smashed="yes">
 <attribute name="VALUE" x="297.815" y="146.685" size="1.778" layer="96"/>
-</instance>
-<instance part="SUPPLY1" gate="GND" x="439.42" y="93.98" smashed="yes">
-<attribute name="VALUE" x="437.515" y="90.805" size="1.778" layer="96"/>
 </instance>
 <instance part="SUPPLY3" gate="GND" x="256.54" y="109.22" smashed="yes">
@@
 </instance>
 <instance part="X_3" gate="G$1" x="317.5" y="40.64" smashed="yes"/>
-<instance part="DC2" gate="G$1" x="170.18" y="86.36" smashed="yes">
-<attribute name="NAME" x="160.02" y="92.075" size="1.778" layer="95"/>
-<attribute name="VALUE" x="160.02" y="76.2" size="1.778" layer="96"/>
-</instance>
-<instance part="X_5" gate="G$1" x="154.94" y="78.74" smashed="yes"/>
-<instance part="U5" gate="A" x="193.04" y="88.9" smashed="yes">
-<attribute name="NAME" x="211.1746" y="98.0186" size="2.083" layer="95" ratio="6"/>
-<attribute name="VALUE" x="210.5352" y="95.4786" size="2.083" layer="96" ratio="6"/>
-</instance>
-<instance part="X_8" gate="G$1" x="198.12" y="73.66" smashed="yes"/>
-<instance part="C1" gate="G$1" x="241.3" y="83.82" smashed="yes">
-<attribute name="NAME" x="242.316" y="84.455" size="1.778" layer="95"/>
-<attribute name="VALUE" x="242.316" y="79.629" size="1.778" layer="96"/>
-</instance>
-<instance part="X_7" gate="G$1" x="241.3" y="76.2" smashed="yes"/>
 <instance part="U3" gate="A" x="378.46" y="58.42" smashed="yes">
 <attribute name="NAME" x="365.76" y="72.12" size="2.0828" layer="95" ratio="10" rot="SR0"/>
@@
 <wire x1="317.5" y1="50.8" x2="317.5" y2="40.64" width="0.1524" layer="91"/>
 <pinref part="X_3" gate="G$1" pin="0"/>
-</segment>
-<segment>
-<pinref part="X_5" gate="G$1" pin="0"/>
-<pinref part="DC2" gate="G$1" pin="-VIN"/>
-<wire x1="154.94" y1="78.74" x2="154.94" y2="83.82" width="0.1524" layer="91"/>
-<wire x1="154.94" y1="83.82" x2="157.48" y2="83.82" width="0.1524" layer="91"/>
-</segment>
-<segment>
-<pinref part="DC2" gate="G$1" pin="-VOUT"/>
-<wire x1="182.88" y1="83.82" x2="182.88" y2="78.74" width="0.1524" layer="91"/>
-<wire x1="182.88" y1="78.74" x2="198.12" y2="78.74" width="0.1524" layer="91"/>
-<pinref part="X_8" gate="G$1" pin="0"/>
-<wire x1="198.12" y1="73.66" x2="198.12" y2="78.74" width="0.1524" layer="91"/>
-</segment>
-<segment>
-<pinref part="X_7" gate="G$1" pin="0"/>
-<pinref part="C1" gate="G$1" pin="2"/>
-<wire x1="241.3" y1="76.2" x2="241.3" y2="78.74" width="0.1524" layer="91"/>
 </segment>
 <segment>
@@
 <pinref part="U1" gate="A" pin="VCC"/>
 </segment>
-<segment>
-<pinref part="DC2" gate="G$1" pin="+VOUT"/>
-<wire x1="182.88" y1="88.9" x2="195.58" y2="88.9" width="0.1524" layer="91"/>
-<label x="182.88" y="88.9" size="1.778" layer="95"/>
-<pinref part="U5" gate="A" pin="VCC"/>
-</segment>
 </net>
 <net name="N$2" class="0">
@@
 <pinref part="SUPPLY2" gate="GND" pin="GND"/>
 <wire x1="289.56" y1="152.4" x2="299.72" y2="152.4" width="0.1524" layer="91"/>
-</segment>
-<segment>
-<pinref part="E1" gate="G$1" pin="GND"/>
-<wire x1="444.5" y1="101.6" x2="439.42" y2="101.6" width="0.1524" layer="91"/>
-<pinref part="SUPPLY1" gate="GND" pin="GND"/>
-<wire x1="439.42" y1="101.6" x2="439.42" y2="96.52" width="0.1524" layer="91"/>
 </segment>
 <segment>
@@
 <net name="N$5" class="0">
 <segment>
-<pinref part="E1" gate="G$1" pin="UART_TX"/>
 <wire x1="444.5" y1="132.08" x2="439.42" y2="132.08" width="0.1524" layer="91"/>
 <wire x1="439.42" y1="132.08" x2="439.42" y2="121.92" width="0.1524" layer="91"/>
@@
 <net name="N$7" class="0">
 <segment>
-<pinref part="E1" gate="G$1" pin="UART_RX"/>
 <wire x1="444.5" y1="129.54" x2="441.96" y2="129.54" width="0.1524" layer="91"/>
 <wire x1="441.96" y1="129.54" x2="441.96" y2="119.38" width="0.1524" layer="91"/>
@@
 <wire x1="342.9" y1="50.8" x2="342.9" y2="55.88" width="0.1524" layer="91"/>
 <wire x1="347.98" y1="50.8" x2="347.98" y2="91.44" width="0.1524" layer="91"/>
-<pinref part="U2" gate="A" pin="P2.1/TB0.2"/>
-<wire x1="436.88" y1="114.3" x2="439.42" y2="114.3" width="0.1524" layer="91"/>
-<wire x1="439.42" y1="114.3" x2="439.42" y2="106.68" width="0.1524" layer="91"/>
-<wire x1="439.42" y1="106.68" x2="424.18" y2="106.68" width="0.1524" layer="91"/>
-<wire x1="424.18" y1="106.68" x2="424.18" y2="91.44" width="0.1524" layer="91"/>
-<wire x1="424.18" y1="91.44" x2="408.94" y2="91.44" width="0.1524" layer="91"/>
 <pinref part="U3" gate="A" pin="VOUTA"/>
 <wire x1="408.94" y1="91.44" x2="347.98" y2="91.44" width="0.1524" layer="91"/>
@@
 <wire x1="408.94" y1="63.5" x2="408.94" y2="91.44" width="0.1524" layer="91"/>
 <junction x="408.94" y="91.44"/>
+<wire x1="408.94" y1="91.44" x2="464.82" y2="91.44" width="0.1524" layer="91"/>
+<wire x1="464.82" y1="91.44" x2="464.82" y2="147.32" width="0.1524" layer="91"/>
+<wire x1="464.82" y1="147.32" x2="436.88" y2="147.32" width="0.1524" layer="91"/>
+<wire x1="436.88" y1="147.32" x2="436.88" y2="132.08" width="0.1524" layer="91"/>
+<pinref part="U2" gate="A" pin="P1.2/UCA0RXD/UCA0SOMI/TB0TRG/C2/A2/VEREF-"/>
 </segment>
 </net>
@@
 </segment>
 </net>
-<net name="N$12" class="0">
-<segment>
-<wire x1="236.22" y1="88.9" x2="241.3" y2="88.9" width="0.1524" layer="91"/>
-<label x="238.76" y="91.44" size="1.778" layer="95"/>
-<pinref part="U5" gate="A" pin="OUT"/>
-<pinref part="C1" gate="G$1" pin="1"/>
-<wire x1="241.3" y1="86.36" x2="241.3" y2="88.9" width="0.1524" layer="91"/>
-<junction x="241.3" y="88.9"/>
-<wire x1="241.3" y1="88.9" x2="302.26" y2="88.9" width="0.1524" layer="91"/>
-<pinref part="E1" gate="G$1" pin="+3.3V"/>
-<wire x1="444.5" y1="104.14" x2="302.26" y2="104.14" width="0.1524" layer="91"/>
-<wire x1="302.26" y1="104.14" x2="302.26" y2="88.9" width="0.1524" layer="91"/>
-</segment>
-</net>
 <net name="N$6" class="0">
 <segment>
-<pinref part="DC2" gate="G$1" pin="+VIN"/>
-<wire x1="139.7" y1="88.9" x2="157.48" y2="88.9" width="0.1524" layer="91"/>
 <pinref part="DC1" gate="G$1" pin="+VIN"/>
-<wire x1="116.84" y1="149.86" x2="139.7" y2="149.86" width="0.1524" layer="91"/>
+<wire x1="116.84" y1="149.86" x2="154.94" y2="149.86" width="0.1524" layer="91"/>
 <label x="139.7" y="149.86" size="1.778" layer="95"/>
 <pinref part="BT2" gate="G$1" pin="-"/>
-<wire x1="139.7" y1="149.86" x2="154.94" y2="149.86" width="0.1524" layer="91"/>
 <wire x1="116.84" y1="142.24" x2="116.84" y2="149.86" width="0.1524" layer="91"/>
-<wire x1="139.7" y1="88.9" x2="139.7" y2="149.86" width="0.1524" layer="91"/>
-<junction x="139.7" y="149.86"/>
 </segment>
 </net>
@@
 </segment>
 </net>
+<net name="N$10" class="0">
+<segment>
+<pinref part="U2" gate="A" pin="P2.1/TB0.2"/>
+<wire x1="436.88" y1="114.3" x2="439.42" y2="114.3" width="0.1524" layer="91"/>
+</segment>
+</net>
